Commit message: transmission and control

File: arduinobot_description/urdf/arduinobot.urdf.xacro (robot description, xacro)
@@ -2,4 +2,6 @@
 <!-- source xacro format -->
 <robot xmlns:xacro="http://www.ros.org/wiki/xacro" name="arduinobot">
+    <xacro:include filename="$(find arduinobot_description)/urdf/arduinobot_gazebo.xacro" />
+    <xacro:include filename="$(find arduinobot_description)/urdf/arduinobot_ros2_control.xacro" />
     <xacro:property name="PI" value="3.14159"/>
     <xacro:property name="effort" value="30.0"/>
@@ -13,4 +15,14 @@
                      izz="1.0" />
         </inertial>
+    </xacro:macro>
+    <!-- mechanical transmission connecting model to joint_number -->
+    <xacro:macro name="default_transmission" params="number">
+        <transmission name="transmission_${number}">
+            <plugin>transmission_interface/SimpleTransmission</plugin>
+            <actuator name="motor_${number}" role="actuator1"/>
+            <joint name="joint_${number}" role="joint1">
+                <mechanical_reduction>1.0</mechanical_reduction>
+            </joint>
+        </transmission>
     </xacro:macro>
     <!-- /> = close link on same line -->
@@ -227,3 +239,7 @@
         </sensor>
     </gazebo>
+    <xacro:default_transmission number="1"/>
+    <xacro:default_transmission number="2"/>
+    <xacro:default_transmission number="3"/>
+    <xacro:default_transmission number="4"/>
 </robot>

Commit message: URDF update by Antonio

File: arduinobot_description/urdf/arduinobot.urdf.xacro (robot description, xacro)
@@ -2,12 +2,18 @@
 <!-- source xacro format -->
 <robot xmlns:xacro="http://www.ros.org/wiki/xacro" name="arduinobot">
+    <!-- Load Simulated or Real Hardware Interfaces -->
+    <xacro:arg name="is_sim" default="true"/>
+    <!-- Include Gazebo Parameters -->
     <xacro:include filename="$(find arduinobot_description)/urdf/arduinobot_gazebo.xacro" />
+    <!-- Include ros2_control Plugins -->
     <xacro:include filename="$(find arduinobot_description)/urdf/arduinobot_ros2_control.xacro" />
-    <xacro:property name="PI" value="3.14159"/>
-    <xacro:property name="effort" value="30.0"/>
-    <xacro:property name="velocity" value="10.0"/>
+    <!-- Variable = XACRO Property -->
+    <xacro:property name="PI" value="3.14159265359" />
+    <xacro:property name="effort" value="30.0" />
+    <xacro:property name="velocity" value="10.0" />
     <!-- makro to reuse code, option to use params like function -->
-    <xacro:macro name="default_inertial" params="mass" >
+    <xacro:macro name="default_inertial" params="mass">
         <inertial>
+            <origin xyz="0 0 0" rpy="0 0 0"/>
             <mass value="${mass}" />
             <inertia ixx="1.0" ixy="0.0" ixz="0.0"
@@ -21,222 +27,195 @@
             <plugin>transmission_interface/SimpleTransmission</plugin>
             <actuator name="motor_${number}" role="actuator1"/>
-            <joint name="joint_${number}" role="joint1">
+            <joint name="joint_${number}"    role="joint1">
                 <mechanical_reduction>1.0</mechanical_reduction>
             </joint>
         </transmission>
     </xacro:macro>
-    <!-- /> = close link on same line -->
-    <!-- this link is parent of all other links and is interface to outside world-->
+    <!-- link origin = move part only, coordinate system remains unchanged      -->
+    <!-- joint origin = move part and its coordinate system -->
+    <!-- Links, /> = close on same line -->
+    <!-- parent of all other links and interface to outside world-->
     <link name="world"/>
     <link name="base_link">
-        <!-- makro -->
-        <xacro:default_inertial mass="1.0" />
+        <xacro:default_inertial mass="1.0"/>
         <visual>
             <!-- set initial render orientation and position in [dm] -->
-            <origin rpy="0 0 0" xyz="-0.5 -0.5 0" />
-            <geometry>
-                <mesh filename="package://arduinobot_description/meshes/basement.STL" scale="0.01 0.01 0.01" />
-            </geometry>
-        </visual>
-        <collision>
-            <origin rpy="0 0 0" xyz="-0.5 -0.5 0" />
-            <geometry>
-                <mesh filename="package://arduinobot_description/meshes/basement.STL" scale="0.01 0.01 0.01" />
-            </geometry>
-        </collision>
-    </link>
+            <origin rpy="0 0 0" xyz="-0.5 -0.5 0"/>
+            <geometry>
+                <mesh filename="package://arduinobot_description/meshes/basement.STL" scale="0.01 0.01 0.01"/>
+            </geometry>
+        </visual>
+        <collision>
+            <origin rpy="0 0 0" xyz="-0.5 -0.5 0"/>
+            <geometry>
+                <mesh filename="package://arduinobot_description/meshes/basement.STL" scale="0.01 0.01 0.01"/>
+            </geometry>
+        </collision>
+    </link>
+    <link name="base_plate">
+        <xacro:default_inertial mass="0.1"/>
+        <visual>
+            <origin rpy="0 0 0" xyz="-0.39 -0.39 -0.56"/>
+            <geometry>
+                <mesh filename="package://arduinobot_description/meshes/base_plate.STL" scale="0.01 0.01 0.01"/>
+            </geometry>
+        </visual>
+        <collision>
+            <origin rpy="0 0 0" xyz="-0.39 -0.39 -0.56"/>
+            <geometry>
+                <mesh filename="package://arduinobot_description/meshes/base_plate.STL" scale="0.01 0.01 0.01"/>
+            </geometry>
+        </collision>
+    </link>
+    <link name="forward_drive_arm">
+        <xacro:default_inertial mass="0.1"/>
+        <visual>
+            <origin rpy=" 0 -${PI / 2} ${PI / 2}" xyz="0.19 0.06 -0.08"/>
+            <geometry>
+                <mesh filename="package://arduinobot_description/meshes/forward_drive_arm.STL" scale="0.01 0.01 0.01"/>
+            </geometry>
+        </visual>
+        <collision>
+            <origin rpy=" 0 -${PI / 2} ${PI / 2}" xyz="0.19 0.06 -0.08"/>
+            <geometry>
+                <mesh filename="package://arduinobot_description/meshes/forward_drive_arm.STL" scale="0.01 0.01 0.01"/>
+            </geometry>
+        </collision>
+    </link>
+    <link name="horizontal_arm">
+        <xacro:default_inertial mass="0.1"/>
+        <visual>
+            <origin rpy="${PI / 2} 0 ${PI / 2}" xyz="-0.03 -0.4 -0.06"/>
+            <geometry>
+                <mesh filename="package://arduinobot_description/meshes/horizontal_arm.STL" scale="0.01 0.01 0.01"/>
+            </geometry>
+        </visual>
+        <collision>
+            <origin rpy="${PI / 2} 0 ${PI / 2}" xyz="-0.03 -0.4 -0.06"/>
+            <geometry>
+                <mesh filename="package://arduinobot_description/meshes/horizontal_arm.STL" scale="0.01 0.01 0.01"/>
+            </geometry>
+        </collision>
+    </link>
+    <link name="claw_support">
+        <xacro:default_inertial mass="0.05"/>
+        <visual>
+            <origin rpy="0 0 ${PI / 2}" xyz="0 -0.05 -0.15"/>
+            <geometry>
+                <mesh filename="package://arduinobot_description/meshes/claw_support.STL" scale="0.01 0.01 0.01"/>
+            </geometry>
+        </visual>
+        <collision>
+            <origin rpy="0 0 ${PI / 2}" xyz="0 -0.05 -0.15"/>
+            <geometry>
+                <mesh filename="package://arduinobot_description/meshes/claw_support.STL" scale="0.01 0.01 0.01"/>
+            </geometry>
+        </collision>
+    </link>
+    <link name="gripper_right">
+        <xacro:default_inertial mass="0.01"/>
+        <visual>
+            <origin rpy="0 0 -${PI / 2}" xyz="-0.1 0.50 -0.1"/>
+            <geometry>
+                <mesh filename="package://arduinobot_description/meshes/right_finger.STL" scale="0.01 0.01 0.01"/>
+            </geometry>
+        </visual>
+        <collision>
+            <origin rpy="0 0 -${PI / 2}" xyz="-0.1 0.50 -0.1"/>
+            <geometry>
+                <mesh filename="package://arduinobot_description/meshes/right_finger.STL" scale="0.01 0.01 0.01"/>
+            </geometry>
+        </collision>
+    </link>
+    <link name="gripper_left">
+        <xacro:default_inertial mass="0.01"/>
+        <visual>
+            <origin rpy="0 0 -${PI / 2}" xyz="-0.04 0.50 -0.1"/>
+            <geometry>
+                <mesh filename="package://arduinobot_description/meshes/left_finger.STL" scale="0.01 0.01 0.01"/>
+            </geometry>
+        </visual>
+        <collision>
+            <origin rpy="0 0 -${PI / 2}" xyz="-0.04 0.50 -0.1"/>
+            <geometry>
+                <mesh filename="package://arduinobot_description/meshes/left_finger.STL" scale="0.01 0.01 0.01"/>
+            </geometry>
+        </collision>
+    </link>
+    <link name="rgb_camera">
+        <xacro:default_inertial mass="0.001"/>
+        <visual>
+            <origin rpy="-1.57 0 -1.57" xyz="-0.1 0.125 0.15"/>
+            <geometry>
+                <mesh filename="package://arduinobot_description/meshes/pi_camera.STL" scale="0.01 0.01 0.01"/>
+            </geometry>
+        </visual>
+        <collision>
+            <origin rpy="-1.57 0 -1.57" xyz="-0.1 0.125 0.15"/>
+            <geometry>
+                <mesh filename="package://arduinobot_description/meshes/pi_camera.STL" scale="0.01 0.01 0.01"/>
+            </geometry>
+        </collision>
+    </link>
+    <!-- Joints -->
     <!-- virtual since only attach to outside world -->
     <joint name="virtual_joint" type="fixed">
-        <parent link="world" />
-        <child link="base_link" />
-        <!-- same orientation -->
-        <origin rpy="0 0 0" xyz="0 0 0" />
-    </joint>
-    <link name="base_plate">
-        <xacro:default_inertial mass="0.1" />
-        <visual>
-            <origin rpy="0 0 0" xyz="-0.39 -0.39 -0.56" />
-            <geometry>
-                <mesh filename="package://arduinobot_description/meshes/base_plate.STL" scale="0.01 0.01 0.01" />
-            </geometry>
-        </visual>
-        <collision>
-            <origin rpy="0 0 0" xyz="-0.39 -0.39 -0.56" />
-            <geometry>
-                <mesh filename="package://arduinobot_description/meshes/base_plate.STL" scale="0.01 0.01 0.01" />
-            </geometry>
-        </collision>
-    </link>
-    <joint name="joint_1" type="revolute">
+        <parent link="world"/>
+        <child link="base_link"/>
+        <origin xyz="0 0 0" rpy="0 0 0"/>
+    </joint>
+    <joint name ="joint_1" type="revolute">
         <parent link="base_link"/>
-        <child link="base_plate"/>
+        <child link = "base_plate"/>
+        <origin xyz="0 0 0.307"/>
         <axis xyz="0 0 1"/>
-        <origin rpy="0 0 0" xyz="0 0 0.307" />
-        <limit lower="-${PI/2}" upper="${PI/2}" effort="${effort}" velocity="${velocity}" />
-    </joint>
-    <link name="forward_drive_arm" >
-        <xacro:default_inertial mass="0.1" />
-        <visual>
-            <origin rpy="0 -${PI/2} ${PI/2}" xyz="0.19 0.06 -0.08" />
-            <geometry>
-                <mesh filename="package://arduinobot_description/meshes/forward_drive_arm.STL" scale="0.01 0.01 0.01" />
-            </geometry>
-        </visual>
-        <collision>
-            <origin rpy="0 -${PI/2} ${PI/2}" xyz="0.19 0.06 -0.08" />
-            <geometry>
-                <mesh filename="package://arduinobot_description/meshes/forward_drive_arm.STL" scale="0.01 0.01 0.01" />
-            </geometry>
-        </collision>
-    </link>
-    <joint name="joint_2" type="revolute" >
-        <parent link="base_plate" />
-        <child link="forward_drive_arm" />
-        <axis xyz="1 0 0" />
-        <origin rpy="0 0 0" xyz="-0.02 0 0.35" />
-        <limit lower="-${PI/2}" upper="${PI/2}" effort="${effort}" velocity="${velocity}" />
-    </joint>
-    <link name="horizontal_arm">
-        <xacro:default_inertial mass="0.1" />
-        <visual>
-            <origin rpy="${PI/2} 0 ${PI/2}" xyz="-0.03 -0.4 -0.06" />
-            <geometry>
-                <mesh filename="package://arduinobot_description/meshes/horizontal_arm.STL" scale="0.01 0.01 0.01" />
-            </geometry>
-        </visual>
-        <collision>
-            <origin rpy="${PI/2} 0 ${PI/2}" xyz="-0.03 -0.4 -0.06" />
-            <geometry>
-                <mesh filename="package://arduinobot_description/meshes/horizontal_arm.STL" scale="0.01 0.01 0.01" />
-            </geometry>
-        </collision>
-    </link>
-    <joint name="joint_3" type="revolute" >
-        <parent link="forward_drive_arm" />
-        <child link="horizontal_arm" />
-        <axis xyz="1 0 0" />
-        <origin rpy="0 0 0" xyz="0 0 0.8" />
-        <limit lower="-${PI/2}" upper="${PI/2}" effort="${effort}" velocity="${velocity}" />
-    </joint>
-    <link name="claw_support" >
-        <xacro:default_inertial mass="0.05" />
-        <visual>
-            <origin rpy="0 0 ${PI/2}" xyz="0 -0.05 -0.15" />
-            <geometry>
-                <mesh filename="package://arduinobot_description/meshes/claw_support.STL" scale="0.01 0.01 0.01" />
-            </geometry>
-        </visual>
-        <collision>
-            <origin rpy="0 0 ${PI/2}" xyz="0 -0.05 -0.15" />
-            <geometry>
-                <mesh filename="package://arduinobot_description/meshes/claw_support.STL" scale="0.01 0.01 0.01" />
-            </geometry>
-        </collision>
-    </link>
-    <joint name="horizontal_arm_to_claw_support" type="fixed">
+        <limit lower="-${PI / 2}" upper="${PI / 2}"
+               effort="${effort}" velocity="${velocity}"/>
+    </joint>
+    <joint name ="joint_2" type="revolute">
+        <parent link="base_plate"/>
+        <child link = "forward_drive_arm"/>
+        <origin xyz="-0.02 0 0.35"/>
+        <axis xyz="1 0 0"/>
+        <limit lower="-${PI / 2}" upper="${PI / 2}"
+                effort="${effort}" velocity="${velocity}"/>
+    </joint>
+    <joint name ="joint_3" type="revolute">
+        <parent link="forward_drive_arm"/>
+        <child link = "horizontal_arm"/>
+        <origin xyz="0 0 0.8"/>
+        <axis xyz="1 0 0"/>
+        <limit lower="-${PI / 2}" upper="${PI / 2}"
+               effort="${effort}" velocity="${velocity}"/>
+    </joint>
+    <joint name ="horizontal_arm_to_claw_support" type="fixed">
         <parent link="horizontal_arm"/>
-        <child link="claw_support"/>
-        <origin xyz="0 0.82 0" rpy="0 0 0" />
-    </joint>
-    <link name="gripper_right" >
-        <xacro:default_inertial mass="0.01" />
-        <visual>
-            <origin xyz="-0.1 0.5 -0.1" rpy="0 0 -${PI/2}" />
-            <geometry>
-                <mesh filename="package://arduinobot_description/meshes/right_finger.STL" scale="0.01 0.01 0.01"/>
-            </geometry>
-        </visual>
-        <collision>
-            <origin xyz="-0.1 0.5 -0.1" rpy="0 0 -${PI/2}" />
-            <geometry>
-                <mesh filename="package://arduinobot_description/meshes/right_finger.STL" scale="0.01 0.01 0.01"/>
-            </geometry>
-        </collision>
-    </link>
-    <link name="gripper_left" >
-        <xacro:default_inertial mass="0.01" />
-        <visual>
-            <origin xyz="-0.04 0.5 -0.1" rpy="0 0 -${PI/2}" />
-            <geometry>
-                <mesh filename="package://arduinobot_description/meshes/left_finger.STL" scale="0.01 0.01 0.01"/>
-            </geometry>
-        </visual>
-        <collision>
-            <origin xyz="-0.04 0.5 -0.1" rpy="0 0 -${PI/2}" />
-            <geometry>
-                <mesh filename="package://arduinobot_description/meshes/left_finger.STL" scale="0.01 0.01 0.01"/>
-            </geometry>
-        </collision>
-    </link>
-    <joint name="joint_4" type="revolute">
-        <parent link="claw_support" />
-        <child link="gripper_right"/>
-        <axis xyz="0 0 1" />
-        <origin rpy="0 0 0" xyz="-0.04 0.13 -0.1" />
-        <limit lower="-${PI/2}" upper="0.0" effort="${effort}" velocity="${velocity}" />
-    </joint>
-    <joint name="joint_5" type="revolute">
-        <parent link="claw_support" />
-        <child link="gripper_left"/>
-        <axis xyz="0 0 1" />
-        <origin rpy="0 0 0" xyz="-0.22 0.13 -0.1" />
+        <child link = "claw_support"/>
+        <origin xyz="0 0.82 0"/>
+    </joint>
+    <joint name ="joint_4" type="revolute">
+        <parent link="claw_support"/>
+        <child link = "gripper_right"/>
+        <origin xyz="-0.04 0.13 -0.1"/>
+        <axis xyz="0 0 1"/>
+        <limit lower="-${PI / 2}" upper="0.0"
+               effort="${effort}" velocity="${velocity}"/>
+    </joint>
+    <joint name ="joint_5" type="revolute">
+        <parent link="claw_support"/>
+        <child link = "gripper_left"/>
+        <origin xyz="-0.22 0.13 -0.1"/>
+        <axis xyz="0 0 1"/>
+        <limit lower="0.0" upper="${PI / 2}"
+               effort="${effort}" velocity="${velocity}"/>
         <!-- mimic to ensure symmetrical claw opening -->
-        <mimic joint="joint_4" multiplier="-1" />
-        <limit lower="0.0" upper="${PI/2}" effort="${effort}" velocity="${velocity}" />
-    </joint>
-    <!-- link origin = move part only, coordinate system remains unchanged      -->
-    <link name="rgb_camera" >
-        <xacro:default_inertial mass="0.001" />
-        <visual>
-            <origin xyz="-0.1 0.125 0.15" rpy="-${PI/2} 0 -${PI/2}" />
-            <geometry>
-                <mesh filename="package://arduinobot_description/meshes/pi_camera.STL" scale="0.01 0.01 0.01" />
-            </geometry>
-        </visual>
-        <collision>
-            <origin xyz="-0.1 0.125 0.15" rpy="-${PI/2} 0 -${PI/2}" />
-            <geometry>
-                <mesh filename="package://arduinobot_description/meshes/pi_camera.STL" scale="0.01 0.01 0.01" />
-            </geometry>
-        </collision>
-    </link>
-    <!-- joint origin = move part and its coordinate system -->
-    <joint name="rgb_camera_joint" type="fixed">
+        <mimic joint="joint_4" multiplier="-1"/>
+    </joint>
+    <joint name ="rgb_camera_joint" type="fixed">
         <parent link="base_link"/>
-        <child link="rgb_camera"/>
-        <origin xyz="0 0.45 0.2" rpy="0 -0.5 ${PI/2}" />
-    </joint>
-    <gazebo reference="rgb_camera">
-        <sensor type="camera" name="rgb_camera">
-            <always_on>true</always_on>
-            <update_rate>30.0</update_rate>
-            <camera name="rgb_camera">
-                <horizontal_fov>1.15</horizontal_fov>
-                <vertical_fov>0.71</vertical_fov>
-                <image>
-                    <width>2304</width>
-                    <height>1296</height>
-                    <format>R8G8B8</format>
-                </image>
-                <distortion>
-                    <k1>0.0</k1>
-                    <k2>0.0</k2>
-                    <k3>0.0</k3>
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
File: arduinobot_description/urdf/arduinobot_gazebo.xacro (robot description, xacro)
@@ -1,10 +1,43 @@
 <?xml version="1.0"?>
 <robot xmlns:xacro="http://www.ros.org/wiki/xacro" name="arduinobot">
+    <!-- Gazebo ros2_control plugin -->
     <gazebo>
-        <plugin filename="libgazebo_ros2_control.so" name="gazebo_ros2_control">
-            <robot_param>robot_description</robot_param>
-            <robot_param_node>robot_state_publisher</robot_param_node>
-            <parameters>$(find arduinobot_controller)/config/arduinobot_controllers.yaml</parameters>
-        </plugin>
+      <plugin filename="libgazebo_ros2_control.so" name="gazebo_ros2_control">
+        <robot_param>robot_description</robot_param>
+        <robot_param_node>robot_state_publisher</robot_param_node>
+        <parameters>$(find arduinobot_controller)/config/arduinobot_controllers.yaml</parameters>
+      </plugin>
     </gazebo>
+    <gazebo reference="rgb_camera">
+        <sensor type="camera" name="rgb_camera">
+            <always_on>true</always_on>
+            <update_rate>30.0</update_rate>
+            <camera name="rgb_camera">
+                <horizontal_fov>1.15</horizontal_fov>
+                <vertical_fov>0.71</vertical_fov>
+                <image>
+                    <width>2304</width>
+                    <height>1296</height>
+                    <format>R8G8B8</format>
+                </image>
+                <distortion>
+                    <k1>0.0</k1>
+                    <k2>0.0</k2>
+                    <k3>0.0</k3>
+                    <p1>0.0</p1>
+                    <p2>0.0</p2>
+                    <center>0.5 0.5</center>
+                </distortion>
+            </camera>
+            <plugin name="plugin_name" filename="libgazebo_ros_camera.so">
+                <ros>
+                    <remapping>~/image_raw:=image_raw</remapping>
+                    <remapping>~/camera_info:=camera_info</remapping>
+                </ros>
+                <camera_name>rgb_camera</camera_name>
+                <frame_name>rgb_camera</frame_name>
+                <hack_baseline>0.2</hack_baseline>
+            </plugin>
+        </sensor>
+      </gazebo>
 </robot>
